File: design_files/ASL2001.brd (EAGLE design)
At the start: 12.5 x 12.5 mm, 12 parts, among them U1 DRV8837

Commit message: update format
Parts:
- moved U$5 7.88 mm to (23.9, 20.0), flipped to the bottom
- moved U$9 7.88 mm to (16.1, 20.0), flipped to the bottom
- moved U$11 5.56 mm to (22.8, 17.2), flipped to the bottom
- moved U$2 5.56 mm to (17.2, 22.8), flipped to the bottom
- moved U$3 5.56 mm to (17.2, 17.2), flipped to the bottom
- moved U$4 5.56 mm to (22.8, 22.8), flipped to the bottom
- moved C1 2.50 mm to (18.8, 21.1), flipped to the top
- moved U1 2.22 mm to (21.1, 20.1), flipped to the top
- moved C2 1.62 mm to (19.2, 19.4), flipped to the top
- flipped U$10 to the bottom
- flipped U$8 to the bottom
Other:
- board text added: "2"
- board text added: "2001-3"
- board text removed: "1"
- board text removed: "2001-1"
